Commit message: Rebase from 'upstream'

File: turtlebot_description/urdf/sensors/asus_xtion_pro.urdf.xacro (robot description, xacro)
@@ -15,13 +15,5 @@
       <child link="camera_rgb_frame" />
     </joint>
-    <link name="camera_rgb_frame">
-      <inertial>
-        <mass value="0.001" />
-        <origin xyz="0 0 0" />
-        <inertia ixx="0.0001" ixy="0.0" ixz="0.0"
-          iyy="0.0001" iyz="0.0"
-          izz="0.0001" />
-      </inertial>
-    </link>
+    <link name="camera_rgb_frame"/>
     <joint name="camera_rgb_optical_joint" type="fixed">
       <origin xyz="0 0 0" rpy="${-M_PI/2} 0 ${-M_PI/2}" />
@@ -29,13 +21,5 @@
       <child link="camera_rgb_optical_frame" />
     </joint>
-    <link name="camera_rgb_optical_frame">
-      <inertial>
-        <mass value="0.001" />
-        <origin xyz="0 0 0" />
-        <inertia ixx="0.0001" ixy="0.0" ixz="0.0"
-          iyy="0.0001" iyz="0.0"
-          izz="0.0001" />
-      </inertial>
-    </link>
+    <link name="camera_rgb_optical_frame"/>
     <joint name="camera_joint" type="fixed">
       <origin xyz="0 ${asus_xtion_pro_cam_rel_rgb_py} 0"
@@ -54,13 +38,13 @@
         <origin xyz="0.0 0.0 0.0" rpy="0 0 0" />
         <geometry>
-        <box size="0.0730 .2760 0.0720"/>
+        <box size="0.0730 0.2760 0.0720"/>
       </geometry>
       </collision>
       <inertial>
-        <mass value="0.01" />
+        <mass value="0.170" />
         <origin xyz="0 0 0" />
-        <inertia ixx="0.001" ixy="0.0" ixz="0.0"
-          iyy="0.001" iyz="0.0"
-          izz="0.001" />
+        <inertia ixx="0.001152600" ixy="0.0" ixz="0.0"
+                 iyy="0.000148934" iyz="0.0"
+                 izz="0.001154654" />
       </inertial>
     </link>
@@ -70,13 +54,5 @@
       <child link="camera_depth_frame" />
     </joint>
-    <link name="camera_depth_frame">
-      <inertial>
-        <mass value="0.01" />
-        <origin xyz="0 0 0" />
-        <inertia ixx="0.001" ixy="0.0" ixz="0.0"
-          iyy="0.001" iyz="0.0"
-          izz="0.001" />
-      </inertial>
-    </link>
+    <link name="camera_depth_frame"/>
     <joint name="camera_depth_optical_joint" type="fixed">
       <origin xyz="0 0 0" rpy="${-M_PI/2} 0 ${-M_PI/2}" />
@@ -84,15 +60,7 @@
       <child link="camera_depth_optical_frame" />
     </joint>
-    <link name="camera_depth_optical_frame">
-      <inertial>
-        <mass value="0.001" />
-        <origin xyz="0 0 0" />
-        <inertia ixx="0.0001" ixy="0.0" ixz="0.0"
-          iyy="0.0001" iyz="0.0"
-          izz="0.0001" />
-      </inertial>
-    </link>
-  <!-- RGBD sensor for simulation, same as Kinect -->
-  <turtlebot_sim_3dsensor/>
+    <link name="camera_depth_optical_frame"/>
+    <!-- RGBD sensor for simulation, same as Kinect -->
+    <turtlebot_sim_3dsensor/>
   </xacro:macro>
 </robot>

File: turtlebot_description/urdf/sensors/kinect.urdf.xacro (robot description, xacro)
@@ -10,13 +10,5 @@
       <child link="camera_rgb_frame" />
     </joint>
-    <link name="camera_rgb_frame">
-      <inertial>
-        <mass value="0.001" />
-        <origin xyz="0 0 0" />
-        <inertia ixx="0.0001" ixy="0.0" ixz="0.0"
-                 iyy="0.0001" iyz="0.0"
-                 izz="0.0001" />
-      </inertial>
-    </link>
+    <link name="camera_rgb_frame"/>
     <joint name="camera_rgb_optical_joint" type="fixed">
       <origin xyz="0 0 0" rpy="${-M_PI/2} 0 ${-M_PI/2}" />
@@ -24,42 +16,34 @@
       <child link="camera_rgb_optical_frame" />
     </joint>
-    <link name="camera_rgb_optical_frame">
+    <link name="camera_rgb_optical_frame"/>
+    <joint name="camera_joint" type="fixed">
+      <origin xyz="-0.031 ${-cam_py} -0.016" rpy="0 0 0"/>
+      <parent link="camera_rgb_frame"/>
+      <child link="camera_link"/>
+    </joint>
+      <link name="camera_link">
+      <visual>
+       <origin xyz="0 0 0" rpy="0 0 ${M_PI/2}"/>
+        <geometry>
+         <mesh filename="package://turtlebot_description/meshes/sensors/kinect.dae"/>
+        </geometry>
+      </visual>
+  	  <collision>
+        <origin xyz="0.0 0.0 0.0" rpy="0 0 0"/>
+  	    <geometry>
+  	      <box size="0.07271 0.27794 0.073"/>
+  	    </geometry>
+  	  </collision>
       <inertial>
-        <mass value="0.001" />
+        <mass value="0.564" />
         <origin xyz="0 0 0" />
-        <inertia ixx="0.0001" ixy="0.0" ixz="0.0"
-                 iyy="0.0001" iyz="0.0"
-                 izz="0.0001" />
+        <inertia ixx="0.003881243" ixy="0.0" ixz="0.0"
+                 iyy="0.000498940" iyz="0.0"
+                 izz="0.003879257" />
       </inertial>
     </link>
-  <joint name="camera_joint" type="fixed">
-    <origin xyz="-0.031 ${-cam_py} -0.016" rpy="0 0 0"/>
-    <parent link="camera_rgb_frame"/>
-    <child link="camera_link"/>
-  </joint>
-    <link name="camera_link">
-    <visual>
-     <origin xyz="0 0 0" rpy="0 0 ${M_PI/2}"/>
-      <geometry>
-       <mesh filename="package://turtlebot_description/meshes/sensors/kinect.dae"/>
-      </geometry>
-    </visual>
-	  <collision>
-      <origin xyz="0.0 0.0 0.0" rpy="0 0 0"/>
-	    <geometry>
-	      <box size="0.07271 0.27794 0.073"/>
-	    </geometry>
-	  </collision>
-    <inertial>
-      <mass value="0.001" />
-      <origin xyz="0 0 0" />
-      <inertia ixx="0.0001" ixy="0.0" ixz="0.0"
-               iyy="0.0001" iyz="0.0"
-               izz="0.0001" />
-    </inertial>
-  </link>
-  <!-- The fixed joints & links below are usually published by static_transformers launched by the OpenNi launch
-       files. However, for Gazebo simulation we need them, so we add them here.
-       (Hence, don't publish them additionally!) -->
+    <!-- The fixed joints & links below are usually published by static_transformers launched by the OpenNi launch
+         files. However, for Gazebo simulation we need them, so we add them here.
+         (Hence, don't publish them additionally!) -->
 	<joint name="camera_depth_joint" type="fixed">
 	  <origin xyz="0 ${2 * -cam_py} 0" rpy="0 0 0" />
@@ -67,13 +51,5 @@
 	  <child link="camera_depth_frame" />
 	</joint>
-	<link name="camera_depth_frame">
-    <inertial>
-      <mass value="0.001" />
-      <origin xyz="0 0 0" />
-      <inertia ixx="0.0001" ixy="0.0" ixz="0.0"
-               iyy="0.0001" iyz="0.0"
-               izz="0.0001" />
-    </inertial>
-	</link>
+	<link name="camera_depth_frame"/>
 	<joint name="camera_depth_optical_joint" type="fixed">
 	  <origin xyz="0 0 0" rpy="${-M_PI/2} 0 ${-M_PI/2}" />
@@ -81,13 +57,5 @@
 	  <child link="camera_depth_optical_frame" />
 	</joint>
-	<link name="camera_depth_optical_frame">
-    <inertial>
-      <mass value="0.001" />
-      <origin xyz="0 0 0" />
-      <inertia ixx="0.0001" ixy="0.0" ixz="0.0"
-               iyy="0.0001" iyz="0.0"
-               izz="0.0001" />
-    </inertial>
-	</link>
+	<link name="camera_depth_optical_frame"/>
 	<!-- Kinect sensor for simulation -->
 	<turtlebot_sim_3dsensor/>

File: turtlebot_description/urdf/stacks/hexagons.urdf.xacro (robot description, xacro)
@@ -25,13 +25,13 @@
         <origin xyz="0 0 0" rpy="0 0 0"/>
         <geometry>
-          <cylinder length="0.0492" radius=".006"/>
-        </geometry>
-      </collision>
-      <inertial>
-        <mass value="0.001"/>
-        <origin xyz="0 0 0" rpy="0 0 0"/>
-        <inertia ixx="0.0001" ixy="0.0" ixz="0.0"
-                 iyy="0.0001" iyz="0.0"
-                 izz="0.0001"/>
+          <cylinder length="0.0492" radius="0.006"/>
+        </geometry>
+      </collision>
+      <inertial>
+        <mass value="0.008"/>
+        <origin xyz="0 0 0" rpy="0 0 0"/>
+        <inertia ixx="0.000001686" ixy="0.0" ixz="0.0"
+                 iyy="0.000001686" iyz="0.0"
+                 izz="0.000000144"/>
       </inertial>
     </link>
@@ -53,13 +53,13 @@
         <origin xyz="0 0 0" rpy="0 0 0"/>
         <geometry>
-          <cylinder length="0.0608" radius=".006"/>
-        </geometry>
-      </collision>
-      <inertial>
-        <mass value="0.001"/>
-        <origin xyz="0 0 0"/>
-        <inertia ixx="0.0001" ixy="0.0" ixz="0.0"
-                 iyy="0.0001" iyz="0.0"
-                 izz="0.0001"/>
+          <cylinder length="0.0608" radius="0.006"/>
+        </geometry>
+      </collision>
+      <inertial>
+        <mass value="0.012"/>
+        <origin xyz="0 0 0"/>
+        <inertia ixx="0.000003805" ixy="0.0" ixz="0.0"
+                 iyy="0.000003805" iyz="0.0"
+                 izz="0.000000216"/>
       </inertial>
     </link>
@@ -81,13 +81,13 @@
         <origin xyz="0 0 0" rpy="0 0 0"/>
         <geometry>
-          <cylinder length="0.2032" radius=".006"/>
-        </geometry>
-      </collision>
-      <inertial>
-        <mass value="0.001"/>
-        <origin xyz="0 0 0"/>
-        <inertia ixx="0.0001" ixy="0.0" ixz="0.0"
-                 iyy="0.0001" iyz="0.0"
-                 izz="0.0001"/>
+          <cylinder length="0.2032" radius="0.006"/>
+        </geometry>
+      </collision>
+      <inertial>
+        <mass value="0.060"/>
+        <origin xyz="0 0 0"/>
+        <inertia ixx="0.000206991" ixy="0.0" ixz="0.0"
+                 iyy="0.000206991" iyz="0.0"
+                 izz="0.000001080"/>
       </inertial>
     </link>
@@ -102,5 +102,4 @@
       <visual>
         <origin xyz="0 0 0" rpy="0 0 0"/>
-<!--         <origin xyz="0 0 0" rpy="${-M_PI/2} ${M_PI} 0"/> -->
         <geometry>
           <mesh filename="package://turtlebot_description/meshes/stacks/hexagons/pole_kinect.dae"/>
@@ -114,9 +113,9 @@
       </collision>
       <inertial>
-        <mass value="0.001"/>
-        <origin xyz="0 0 0"/>
-        <inertia ixx="0.0001" ixy="0.0" ixz="0.0"
-                 iyy="0.0001" iyz="0.0"
-                 izz="0.0001"/>
+        <mass value="0.020"/>
+        <origin xyz="0 0 0"/>
+        <inertia ixx="0.000014782" ixy="0.0" ixz="0.0"
+                 iyy="0.000014782" iyz="0.0"
+                 izz="0.000000360"/>
       </inertial>
     </link>
@@ -153,9 +152,9 @@
       </collision>
       <inertial>
-        <mass value="0.01" />
+        <mass value="0.520" />
         <origin xyz="0 0 0" />
-        <inertia ixx="0.01" ixy="0.0" ixz="0.0"
-                 iyy="0.01" iyz="0.0"
-                 izz="0.01" />
+        <inertia ixx="0.003328" ixy="0.0" ixz="0.0"
+                 iyy="0.003328" iyz="0.0"
+                 izz="0.006656" />
       </inertial>
     </link>
@@ -183,9 +182,9 @@
       </collision>
       <inertial>
-        <mass value="0.01" />
+        <mass value="0.520" />
         <origin xyz="0 0 0" />
-        <inertia ixx="0.01" ixy="0.0" ixz="0.0"
-                 iyy="0.01" iyz="0.0"
-                 izz="0.01" />
+        <inertia ixx="0.003328" ixy="0.0" ixz="0.0"
+                 iyy="0.003328" iyz="0.0"
+                 izz="0.006656" />
       </inertial>
     </link>
@@ -215,9 +214,9 @@
       </collision>
       <inertial>
-        <mass value="0.01"/>
-        <origin xyz="0 0 0"/>
-        <inertia ixx="0.01" ixy="0.0" ixz="0.0"
-                 iyy="0.01" iyz="0.0"
-                 izz="0.01" />
+        <mass value="0.520"/>
+        <origin xyz="0 0 0"/>
+        <inertia ixx="0.003328" ixy="0.0" ixz="0.0"
+                 iyy="0.003328" iyz="0.0"
+                 izz="0.006656" />
       </inertial>
     </link>
